Commit message: Add - Robot on Gazebo

File: frcobot_description/urdf/fr3_gazebo.xacro (robot description, xacro)
@@ -1,3 +1,2 @@
-<?xml version="1.0" encoding="utf-8" ?>
 <!-- This URDF was automatically created by SolidWorks to URDF Exporter! Originally created by Stephen Brawner (brawner@gmail.com)
      Commit Version: 1.5.1-0-g916b5db  Build Version: 1.5.7152.31018

File: frcobot_description/urdf/fr3_robot.xacro (robot description, xacro)
@@ -1,6 +1,2 @@
-<?xml version="1.0" encoding="utf-8"?>
-<!-- This URDF was automatically created by SolidWorks to URDF Exporter! Originally created by Stephen Brawner (brawner@gmail.com)
-     Commit Version: 1.5.1-0-g916b5db  Build Version: 1.5.7152.31018
-     For more information, please see http://wiki.ros.org/sw_urdf_exporter -->
 <robot
   name="fr3_robot_v_5_0">
@@ -33,5 +29,5 @@
       <geometry>
         <mesh
-          filename="package://frcobot_description/meshes/fr3/visual/base_link.DAE" />
+          filename="/home/siw/ws/src/frcobot_ros2/frcobot_description/meshes/fr3/visual/base_link.DAE" />
       </geometry>
       <material
@@ -47,5 +43,5 @@
       <geometry>
         <mesh
-          filename="package://frcobot_description/meshes/fr3/collision/base_link.STL" />
+          filename="/home/siw/ws/src/frcobot_ros2/frcobot_description/meshes/fr3/collision/base_link.STL" />
       </geometry>
     </collision>
@@ -73,19 +69,19 @@
       <geometry>
         <mesh
-          filename="package://frcobot_description/meshes/fr3/visual/shoulder_Link.DAE" />
-      </geometry>
-      <material
-        name="">
-        <color
-          rgba="0.898039215686275 0.917647058823529 0.929411764705882 1" />
-      </material>
-    </visual>
-    <collision>
-      <origin
-        xyz="0 0 0"
-        rpy="0 0 0" />
-      <geometry>
-        <mesh
-          filename="package://frcobot_description/meshes/fr3/collision/shoulder_Link.STL" />
+          filename="/home/siw/ws/src/frcobot_ros2/frcobot_description/meshes/fr3/visual/shoulder_Link.DAE" />
+      </geometry>
+      <material
+        name="">
+        <color
+          rgba="0.898039215686275 0.917647058823529 0.929411764705882 1" />
+      </material>
+    </visual>
+    <collision>
+      <origin
+        xyz="0 0 0"
+        rpy="0 0 0" />
+      <geometry>
+        <mesh
+          filename="/home/siw/ws/src/frcobot_ros2/frcobot_description/meshes/fr3/collision/shoulder_Link.STL" />
       </geometry>
     </collision>
@@ -145,19 +141,19 @@
       <geometry>
         <mesh
-          filename="package://frcobot_description/meshes/fr3/visual/upperarm_Link.DAE" />
-      </geometry>
-      <material
-        name="">
-        <color
-          rgba="0.898039215686275 0.917647058823529 0.929411764705882 1" />
-      </material>
-    </visual>
-    <collision>
-      <origin
-        xyz="0 0 0"
-        rpy="0 0 0" />
-      <geometry>
-        <mesh
-          filename="package://frcobot_description/meshes/fr3/collision/upperarm_Link.STL" />
+          filename="/home/siw/ws/src/frcobot_ros2/frcobot_description/meshes/fr3/visual/upperarm_Link.DAE" />
+      </geometry>
+      <material
+        name="">
+        <color
+          rgba="0.898039215686275 0.917647058823529 0.929411764705882 1" />
+      </material>
+    </visual>
+    <collision>
+      <origin
+        xyz="0 0 0"
+        rpy="0 0 0" />
+      <geometry>
+        <mesh
+          filename="/home/siw/ws/src/frcobot_ros2/frcobot_description/meshes/fr3/collision/upperarm_Link.STL" />
       </geometry>
     </collision>
@@ -214,19 +210,19 @@
       <geometry>
         <mesh
-          filename="package://frcobot_description/meshes/fr3/visual/forearm_Link.DAE" />
-      </geometry>
-      <material
-        name="">
-        <color
-          rgba="0.898039215686275 0.917647058823529 0.929411764705882 1" />
-      </material>
-    </visual>
-    <collision>
-      <origin
-        xyz="0 0 0"
-        rpy="0 0 0" />
-      <geometry>
-        <mesh
-          filename="package://frcobot_description/meshes/fr3/collision/forearm_Link.STL" />
+          filename="/home/siw/ws/src/frcobot_ros2/frcobot_description/meshes/fr3/visual/forearm_Link.DAE" />
+      </geometry>
+      <material
+        name="">
+        <color
+          rgba="0.898039215686275 0.917647058823529 0.929411764705882 1" />
+      </material>
+    </visual>
+    <collision>
+      <origin
+        xyz="0 0 0"
+        rpy="0 0 0" />
+      <geometry>
+        <mesh
+          filename="/home/siw/ws/src/frcobot_ros2/frcobot_description/meshes/fr3/collision/forearm_Link.STL" />
       </geometry>
     </collision>
@@ -283,19 +279,19 @@
       <geometry>
         <mesh
-          filename="package://frcobot_description/meshes/fr3/visual/wrist1_Link.DAE" />
-      </geometry>
-      <material
-        name="">
-        <color
-          rgba="0.898039215686275 0.917647058823529 0.929411764705882 1" />
-      </material>
-    </visual>
-    <collision>
-      <origin
-        xyz="0 0 0"
-        rpy="0 0 0" />
-      <geometry>
-        <mesh
-          filename="package://frcobot_description/meshes/fr3/collision/wrist1_Link.STL" />
+          filename="/home/siw/ws/src/frcobot_ros2/frcobot_description/meshes/fr3/visual/wrist1_Link.DAE" />
+      </geometry>
+      <material
+        name="">
+        <color
+          rgba="0.898039215686275 0.917647058823529 0.929411764705882 1" />
+      </material>
+    </visual>
+    <collision>
+      <origin
+        xyz="0 0 0"
+        rpy="0 0 0" />
+      <geometry>
+        <mesh
+          filename="/home/siw/ws/src/frcobot_ros2/frcobot_description/meshes/fr3/collision/wrist1_Link.STL" />
       </geometry>
     </collision>
@@ -352,19 +348,19 @@
       <geometry>
         <mesh
-          filename="package://frcobot_description/meshes/fr3/visual/wrist2_Link.DAE" />
-      </geometry>
-      <material
-        name="">
-        <color
-          rgba="0.898039215686275 0.917647058823529 0.929411764705882 1" />
-      </material>
-    </visual>
-    <collision>
-      <origin
-        xyz="0 0 0"
-        rpy="0 0 0" />
-      <geometry>
-        <mesh
-          filename="package://frcobot_description/meshes/fr3/collision/wrist2_Link.STL" />
+          filename="/home/siw/ws/src/frcobot_ros2/frcobot_description/meshes/fr3/visual/wrist2_Link.DAE" />
+      </geometry>
+      <material
+        name="">
+        <color
+          rgba="0.898039215686275 0.917647058823529 0.929411764705882 1" />
+      </material>
+    </visual>
+    <collision>
+      <origin
+        xyz="0 0 0"
+        rpy="0 0 0" />
+      <geometry>
+        <mesh
+          filename="/home/siw/ws/src/frcobot_ros2/frcobot_description/meshes/fr3/collision/wrist2_Link.STL" />
       </geometry>
     </collision>
@@ -421,19 +417,19 @@
       <geometry>
         <mesh
-          filename="package://frcobot_description/meshes/fr3/visual/wrist3_Link.DAE" />
-      </geometry>
-      <material
-        name="">
-        <color
-          rgba="0.898039215686275 0.917647058823529 0.929411764705882 1" />
-      </material>
-    </visual>
-    <collision>
-      <origin
-        xyz="0 0 0"
-        rpy="0 0 0" />
-      <geometry>
-        <mesh
-          filename="package://frcobot_description/meshes/fr3/collision/wrist3_Link.STL" />
+          filename="/home/siw/ws/src/frcobot_ros2/frcobot_description/meshes/fr3/visual/wrist3_Link.DAE" />
+      </geometry>
+      <material
+        name="">
+        <color
+          rgba="0.898039215686275 0.917647058823529 0.929411764705882 1" />
+      </material>
+    </visual>
+    <collision>
+      <origin
+        xyz="0 0 0"
+        rpy="0 0 0" />
+      <geometry>
+        <mesh
+          filename="/home/siw/ws/src/frcobot_ros2/frcobot_description/meshes/fr3/collision/wrist3_Link.STL" />
       </geometry>
     </collision>
