Commit message: Add meshless flange_Link to FR3WML URDF (#6)
Add a fixed flange frame 10 cm along the wrist3 z-axis with the same
orientation, representing the robot flange without visual or collision
geometry.

Co-authored-by: Cursor Agent <cursoragent@cursor.com>
Co-authored-by: Stanisław Piasecki <Stachq1@users.noreply.github.com>

File: fairino_description/urdf/FR3WML.urdf (robot description, URDF)
Before this commit: robot FR3WML, 7 links, 7 joints
Links:
- added link flange_Link, mass 0.001
Joints:
- removed joint tool
- added joint flange: type fixed, parent wrist3_Link, child flange_Link, origin xyz=0 0 0.1 rpy=0 0 0, axis 0 0 0, limit lower=0 upper=0 effort=0 velocity=0

Commit message: Add approximate RobotDigg TCP and finger frames (#8)
* Add approximate RobotDigg TCP and finger frames

Co-authored-by: Stanisław Piasecki <Stachq1@users.noreply.github.com>

* Refine RobotDigg gripper geometry

Co-authored-by: Stanisław Piasecki <Stachq1@users.noreply.github.com>

* Set open gripper pose and flange twist

Co-authored-by: Stanisław Piasecki <Stachq1@users.noreply.github.com>

* Correct open gripper V geometry

Co-authored-by: Stanisław Piasecki <Stachq1@users.noreply.github.com>

* Shorten fingers and close palm clearance

Co-authored-by: Stanisław Piasecki <Stachq1@users.noreply.github.com>

---------

Co-authored-by: Cursor Agent <cursoragent@cursor.com>
Co-authored-by: Stanisław Piasecki <Stachq1@users.noreply.github.com>

File: fairino_description/urdf/FR3WML.urdf (robot description, URDF)
Before this commit: robot FR3WML, 8 links, 7 joints
Links:
- added link robotdigg_gripper_base; collision box size=0.070 0.090 0.084; visual box size=0.070 0.090 0.084
- added link robotdigg_left_finger; collision box size=0.025 0.012 0.109; visual box size=0.025 0.012 0.109
- added link robotdigg_right_finger; collision box size=0.025 0.012 0.109; visual box size=0.025 0.012 0.109
- added link robotdigg_tcp
Joints:
- added joint robotdigg_gripper_base_joint: type fixed, parent flange_Link, child robotdigg_gripper_base, origin xyz=0 0 0.042 rpy=0 0 0.785398
- added joint robotdigg_left_finger_joint: type fixed, parent robotdigg_gripper_base, child robotdigg_left_finger, origin xyz=0 0.0555814 0.098 rpy=-0.375752 0 0
- added joint robotdigg_right_finger_joint: type fixed, parent robotdigg_gripper_base, child robotdigg_right_finger, origin xyz=0 -0.0555814 0.098 rpy=0.375752 0 0
- added joint robotdigg_tcp_joint: type fixed, parent robotdigg_gripper_base, child robotdigg_tcp, origin xyz=0 0 0.098 rpy=0 0 0
